Commit message: added link_tcp gripper close

File: src/arm_rviz/urdf/skai_arm.urdf (robot description, URDF)
Before this commit: robot skai_arm, 9 links, 8 joints
Links:
- added link link_tcp; visual sphere radius=0.008
Joints:
- added joint tcp_joint: type fixed, parent J_6, child link_tcp, origin xyz=0 0 0 rpy=0 0 0
